File: VoltageRegulationBoard.brd (EAGLE design)
At the start: 65.6 x 53.4 mm, 10 parts, among them T1 MMBT3904LT1GOSCT-ND(SMALL-SIG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, T2 FZT653-NPNBJT

Commit message: Placed Isolated switchin regulator on board
Parts:
- moved U$2 31.4 mm to (-15.2, 26.7), turned to 270 degrees
- moved RREF 9.25 mm to (21.6, 36.8)
- moved REF_POT 8.98 mm to (26.7, 36.8)
Changed lines of the file:
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@@
 <?xml version="1.0" encoding="utf-8"?>
 <!DOCTYPE eagle SYSTEM "eagle.dtd">
-<eagle version="7.4.0">
+<eagle version="7.6.0">
 <drawing>
 <settings>
@@
 </autorouter>
 <elements>
-<element name="REF_POT" library="voltageReg" package="3-THRU" value="POTENTIOMETER" x="17.78" y="35.56"/>
+<element name="REF_POT" library="voltageReg" package="3-THRU" value="POTENTIOMETER" x="26.67" y="36.83"/>
 <element name="RFB1" library="resistor" package="R0603" value="22k" x="22.86" y="13.97"/>
 <element name="RFB2" library="resistor" package="R0603" value="3k" x="19.05" y="13.97"/>
 <element name="RLIMIT" library="resistor" package="R2512" value="1" x="36.83" y="13.97"/>
-<element name="RREF" library="resistor" package="R0603" value="46k" x="12.7" y="34.29" rot="R270"/>
+<element name="RREF" library="resistor" package="R0603" value="46k" x="21.59" y="36.83" rot="R270"/>
 <element name="T1" library="voltageReg" package="SOT23" value="MMBT3904LT1GOSCT-ND(SMALL-SIGNAL-NMOS)" x="33.02" y="19.05" rot="R90"/>
 <element name="T2" library="voltageReg" package="SOT223" value="FZT653-NPNBJT" x="38.1" y="20.32"/>
 <element name="U$1" library="foe-scale" package="SOIC8" value="LMC6482" x="21.59" y="19.05" rot="R90"/>
-<element name="U$2" library="voltageReg" package="REC7.5-1209" value="REC7.5-1209" x="-41.91" y="10.16"/>
+<element name="U$2" library="voltageReg" package="REC7.5-1209" value="REC7.5-1209" x="-15.24" y="26.67" rot="R270"/>
 <element name="U$3" library="voltageReg" package="2-THRU" value="3XJUMPER" x="24.13" y="27.94" rot="R270"/>
 </elements>
@@
 <contactref element="U$2" pad="VIN1+"/>
 <contactref element="U$2" pad="VIN2+"/>
-<wire x1="-36.83" y1="10.16" x2="-39.37" y2="10.16" width="0" layer="19" extent="1-1"/>
+<wire x1="-15.24" y1="21.59" x2="-15.24" y2="24.13" width="0" layer="19" extent="1-1"/>
 </signal>
 <signal name="INST_GND">
 <contactref element="U$2" pad="VIN1-"/>
 <contactref element="U$2" pad="VIN2-"/>
-<wire x1="-36.83" y1="35.77" x2="-39.37" y2="35.77" width="0" layer="19" extent="1-1"/>
+<wire x1="10.37" y1="21.59" x2="10.37" y2="24.13" width="0" layer="19" extent="1-1"/>
 </signal>
 <signal name="9V">
@@
 <wire x1="38.1" y1="20.32" x2="38.1" y2="27.72" width="0" layer="19" extent="1-1"/>
 <wire x1="18.99" y1="17.145" x2="38.1" y2="20.32" width="0" layer="19" extent="1-1"/>
-<wire x1="-16.51" y1="10.16" x2="18.99" y2="17.145" width="0" layer="19" extent="1-1"/>
+<wire x1="-15.24" y1="1.27" x2="18.99" y2="17.145" width="0" layer="19" extent="1-1"/>
 </signal>
 <signal name="GND_ISO">
@@
 <contactref element="REF_POT" pad="3"/>
 <contactref element="REF_POT" pad="2"/>
-<wire x1="20.32" y1="35.56" x2="22.86" y2="35.56" width="0" layer="19" extent="1-1"/>
-<wire x1="24.19" y1="20.955" x2="22.86" y2="35.56" width="0" layer="19" extent="1-1"/>
+<wire x1="29.21" y1="36.83" x2="31.75" y2="36.83" width="0" layer="19" extent="1-1"/>
+<wire x1="24.19" y1="20.955" x2="31.75" y2="36.83" width="0" layer="19" extent="1-1"/>
 <wire x1="18.2" y1="13.97" x2="24.19" y2="20.955" width="0" layer="19" extent="1-1"/>
-<wire x1="-21.59" y1="10.16" x2="18.2" y2="13.97" width="0" layer="19" extent="1-1"/>
+<wire x1="-15.24" y1="6.35" x2="18.2" y2="13.97" width="0" layer="19" extent="1-1"/>
 </signal>
 <signal name="VFB">
@@
 <contactref element="REF_POT" pad="1"/>
 <contactref element="U$3" pad="1A"/>
-<wire x1="12.7" y1="35.14" x2="24.13" y2="27.94" width="0" layer="19" extent="1-1"/>
-<wire x1="17.78" y1="35.56" x2="12.7" y2="35.14" width="0" layer="19" extent="1-1"/>
+<wire x1="21.59" y1="37.68" x2="24.13" y2="27.94" width="0" layer="19" extent="1-1"/>
+<wire x1="26.67" y1="36.83" x2="21.59" y2="37.68" width="0" layer="19" extent="1-1"/>
 </signal>
 <signal name="5V">

Commit message: layout and schematic complete. Ready for final review
Parts:
- removed REF_POT: POTENTIOMETER, voltageReg:3-THRU
- removed RFB1: 22k, resistor:R0603
- removed RFB2: 3k, resistor:R0603
- removed RLIMIT: 1, resistor:R2512
- removed RREF: 46k, resistor:R0603
- added -15V, -9V_U, 5V, 9V_F_S, 9V_UF, GND_ISO, GND_ISO_UF, VREF: TST_PT, voltageReg:TST_POINT
- added C1, C11, C13, C14, C17, C23, C29, C3, C9: 2.2uF, resistor:C0603
- added C10, C12, C15, C16, C2, C22, C26, C30, C4, C8: .01uF, resistor:C0603
- added C18, C21, C27: 22uF, resistor:C1206
- added C19, C28, C5, C6, C7: 0.1uF, resistor:C0603
- added C20, C31: 1uF, resistor:C0603
- added C24: .1uF, resistor:C0603
- added C25: 1000pF, resistor:C0603
- added L1, L2, L3: (no value), resistor:R0603
- added L1_CUK, L2_CUK: 15uH, voltageReg:INDUCTOR_FOOTPRNT
- added R1: 275k, resistor:R0603
- added R10: POTENTIOMETER, voltageReg:3-THRU
- added R11, R12: DNI, resistor:R0603
- added R13, R14: 4.7k, resistor:R0603
- added R2: 100k, resistor:R0603
- added R3: 3k, resistor:R0603
- added R4: 22k, resistor:R0603
- added R5: 1, resistor:R2512
- added R6: 1M, resistor:R0603
- added R7: 63k, resistor:R0603
- added R8: 10k, resistor:R0603
- added R9: 46k, resistor:R0603
- added U$10: SCHOTTKY, voltageReg:SOD-123
- added U$11, U$14: COMMON_MODE_CHOKE, voltageReg:COMM_MODE_CHOKE
- added U$12, U$13, U$15: FEED_THRU_CAP, voltageReg:3-TERM-CAP
- added U$16: 2-THRU, voltageReg:2-THRU-.1
- added U$17: REG102, voltageReg:SOT-23-5
- added U$18, U$19, U$5: 4-OUT, voltageReg:4-THRU
- added U$20: VREF, voltageReg:SOIC8
- added U$4: MCP3425A0T-E, voltageReg:SOT-23-6
- added U$6: DAC_UMAX, voltageReg:8-UMAX
- added U$7: LM2611, voltageReg:SOT-23-5
- moved U$2 65.2 mm to (45.1, 2.03), flipped to the bottom, turned to 0 degrees
- moved T1 27.7 mm to (8.51, 31.9)
- moved T2 25.3 mm to (13.6, 26.7), turned to 90 degrees
- moved U$3 13.5 mm to (32.0, 38.9)
- moved U$1 1.99 mm to (20.1, 17.7)
Connections:
- removed net 15VDC: U$2.VIN1+, U$2.VIN2+
- removed net 9V: T2.2, T2.4, U$1.8, U$2.VOUT+
- removed net REF: U$1.3, U$3.1B, U$3.2B, U$3.3B
- new net +15V: C26.1, C27.1, C28.1, U$18.2, U$2.VIN1+, U$2.VIN2+
- new net -15V: -15V.P$1, U$18.3
- new net -9V_F_DUAL: C14.2, C16.2, C17.2, U$13.IN, U$5.3
- new net -9V_UF: -9V_U.P$1, C18.1, C19.1, L2.1, L2_CUK.1, R7.2
- new net 5V_REF: C29.1, C30.1, C6.1, R12.2, R9.2, U$20.6, U$6.1, VREF.P$1
- new net 9V_F_DUAL: C13.1, C15.1, C17.1, U$12.OUT, U$5.2
- new net 9V_F_SINGLE: 9V_F_S.P$1, C3.1, C31.1, C4.1, T2.2, T2.4, U$1.8, U$15.OUT, U$17.1, U$17.3, U$20.2
- new net 9V_UF: 9V_UF.P$1, C21.1, L1.1, L1_CUK.2, L3.1, U$2.VOUT+, U$7.4, U$7.5
- new net 9V_UF1: C1.1, C2.1, L3.2, U$14.3
- new net D_GND: C25.1, U$19.2
- new net GND_ISO_UF: C1.2, C10.2, C11.2, C12.2, C18.2, C2.2, C21.2, C9.2, GND_ISO_UF.P$1, R8.1, U$10.2, U$14.1, U$2.VOUT-, U$7.2
- new net N$11: C19.2, R7.1, R8.2, U$7.3
- new net N$12: C20.1, L1_CUK.1, U$7.1
- new net N$13: U$11.4, U$12.IN
- new net N$14: U$11.2, U$13.OUT
- new net N$15: C20.2, L2_CUK.2, U$10.1
- new net N$16: C11.1, C12.1, L2.2, U$11.1
- new net N$17: U$14.4, U$15.IN
- new net N$18: R6.1, U$1.3, U$3.1B, U$3.2B, U$3.3B
- new net N$2: R10.1, R9.1
- new net N$5: C22.1, U$17.4
- new net N$6: C10.1, C9.1, L1.2, U$11.3
- new net SCL: R14.1, U$19.3, U$4.3, U$6.3
- new net SDA: R13.1, U$19.4, U$4.4, U$6.4
- new net V_SENSE: C8.1, R1.1, R2.2, U$4.1
- net 5V: now also 5V.P$1, C23.1, C24.1, C5.1, C7.1, R13.2, R14.2, U$17.5, U$4.5, U$6.5, U$6.7; no longer RREF.2
- net GND_ISO: now also C13.2, C14.1, C15.2, C16.1, C22.2, C23.2, C24.2, C25.2, C29.2, C3.2, C30.2, C31.2, C4.2, C5.2, C6.2, C7.2, C8.2, GND_ISO.P$1, R10.3, R11.1, R2.1, R3.1, R6.2, U$12.GND, U$13.GND, U$14.2, U$15.GND, U$16.1, U$17.2, U$20.4, U$4.2, U$4.6, U$5.1, U$5.4, U$6.2, U$6.8; no longer REF_POT.2, REF_POT.3, RFB2.1, U$2.VOUT-
- net INST_GND: now also C26.2, C27.2, C28.2, U$18.1, U$18.4
- net N$3: now also R5.2; no longer RLIMIT.2
- net REF1: now also R10.2; no longer REF_POT.1, RREF.1
- net REF2: now also U$6.6
- net REF3: now also R11.2, R12.1
- net VADJ: now also R1.2, R4.2, R5.1, U$16.2; no longer RFB1.2, RLIMIT.1
- net VFB: now also R3.2, R4.1; no longer RFB1.1, RFB2.2
Routing:
- net GND_ISO_UF: track 0.00 -> 113.9 mm, vias 0 -> 8
- net GND_ISO: track 0.00 -> 109.4 mm, vias 0 -> 11
- net SDA: track 0.00 -> 67.6 mm, vias 0 -> 2
- net INST_GND: track 0.00 -> 66.1 mm, vias 0 -> 2
- net SCL: track 0.00 -> 65.3 mm, vias 0 -> 1
- net 5V: track 0.00 -> 64.3 mm, vias 0 -> 2
- net VADJ: track 0.00 -> 54.1 mm, vias 0 -> 2
- net 5V_REF: track 0.00 -> 50.7 mm, vias 0 -> 3
- net 9V_F_SINGLE: track 0.00 -> 44.4 mm, vias 0 -> 5
- net VFB: track 0.00 -> 42.1 mm
- net N$1: track 0.00 -> 38.7 mm, vias 0 -> 2
- net -9V_UF: track 0.00 -> 36.9 mm
- net -9V_F_DUAL: track 0.00 -> 31.1 mm
- net N$18: track 0.00 -> 30.4 mm, vias 0 -> 2
- net N$13: track 0.00 -> 28.3 mm, vias 0 -> 1
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- added copper zone on layer 15, net 9V_F_SINGLE
- added copper zone on layer 15, net 9V_UF
- added copper zone on layer 2, net GND_ISO
Other:
- board size 65.6 x 53.4 mm -> 66 x 53.4 mm
- board text added: "DATA"
- board text added: "Make sure connector is inserted the appropriate way"
- board text added: "POT"
- board text added: "POWER"
- board text added: "PRE_AMP"
- board text added: "TEC"

Commit message: Layout mostly complete. Making finishing documentation touches:
Parts:
- added DRILEGEND: (no value), drilegend:DRILEGEND
- J1, J2, J3: value 4-OUT -> (none)
- J4: value 2-THRU -> (none)
- T2: value FZT653-NPNBJT -> (none)
- moved VREF 1.27 mm to (31.2, 24.9)
- moved -9V_U 0.76 mm to (14.0, 13.7)
- renumbered L1_CUK to L6, L2_CUK to L7, U$1 to U1, U$11 to L4, U$12 to FC2, U$13 to FC1, U$14 to L5, U$15 to FC3, U$16 to J4, U$17 to U5, U$18 to J1, U$19 to J3, U$2 to U4, U$20 to U3, U$4 to U6, U$5 to J2, U$6 to U2, U$7 to U7
Routing:
- net GND_ISO_UF: track 113.9 -> 106.4 mm, vias 8 -> 7
- net GND_ISO: track 109.4 -> 105.4 mm
- net V_SENSE: track 17.5 -> 20.9 mm
- net 9V_F_SINGLE: track 44.4 -> 42.6 mm
- net 5V_REF: track 50.7 -> 52.3 mm
- net VADJ: track 54.1 -> 55.3 mm
- net 9V_UF: track 25.8 -> 24.6 mm
- net N$1: track 38.7 -> 39.5 mm
- net SDA: track 67.6 -> 68.1 mm
Other:
- board text added: "01-16"
- board text added: "LAYER-STACK"
