File: VoltageRegulationBoard.sch (EAGLE design)
At the start: 10 parts, among them T1 MMBT3904LT1GOSCT-ND(SMALL-SIG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, T2 FZT653-NPNBJT

Commit message: layout and schematic complete. Ready for final review
Parts:
- removed REF_POT: POTENTIOMETER, voltageReg:POTENTIOMETER
- removed RFB1: 22k, resistor:R-US_R0603
- removed RFB2: 3k, resistor:R-US_R0603
- removed RLIMIT: 1, resistor:R-US_R2512
- removed RREF: 46k, resistor:R-US_R0603
- added -15V, -9V_U, 5V, 9V_F_S, 9V_UF, GND_ISO, GND_ISO_UF, VREF: TST_PT, voltageReg:TST_PT
- added C1, C11, C13, C14, C17, C23, C29, C3, C9: 2.2uF, resistor:C-EUC0603
- added C10, C12, C15, C16, C2, C22, C26, C30, C4, C8: .01uF, resistor:C-EUC0603
- added C18, C21, C27: 22uF, resistor:C-EUC1206
- added C19, C28, C5, C6, C7: 0.1uF, resistor:C-EUC0603
- added C20, C31: 1uF, resistor:C-EUC0603
- added C24: .1uF, resistor:C-EUC0603
- added C25: 1000pF, resistor:C-EUC0603
- added L1, L2, L3: (no value), resistor:R-EU_R0603
- added L1_CUK, L2_CUK: 15uH, voltageReg:INDUCTOR
- added R1: 275k, resistor:R-US_R0603
- added R10: POTENTIOMETER, voltageReg:POTENTIOMETER
- added R11, R12: DNI, resistor:R-US_R0603
- added R13, R14: 4.7k, resistor:R-US_R0603
- added R2: 100k, resistor:R-US_R0603
- added R3: 3k, resistor:R-US_R0603
- added R4: 22k, resistor:R-US_R0603
- added R5: 1, resistor:R-US_R2512
- added R6: 1M, resistor:R-US_R0603
- added R7: 63k, resistor:R-US_R0603
- added R8: 10k, resistor:R-US_R0603
- added R9: 46k, resistor:R-US_R0603
- added U$10: SCHOTTKY, voltageReg:SCHOTTKY
- added U$11, U$14: COMMON_MODE_CHOKE, voltageReg:COMMON_MODE_CHOKE
- added U$12, U$13, U$15: FEED_THRU_CAP, voltageReg:FEED_THRU_CAP
- added U$16: 2-THRU, voltageReg:2-THRU
- added U$17: REG102, voltageReg:REG102
- added U$18, U$19, U$5: 4-OUT, voltageReg:4-OUT
- added U$20: VREF, voltageReg:VREF
- added U$4: MCP3425A0T-E, voltageReg:MCP3425A0T-E
- added U$6: DAC_UMAX, voltageReg:DAC_UMAX
- added U$7: LM2611, voltageReg:LM2611
Connections:
- removed net 15VDC: U$2.VIN+
- removed net 9V: T2.C, U$1G$3.V+, U$2.VOUT+
- removed net REF: U$1G$1.AIN+, U$3.COMMON
- new net +15V: C26.1, C27.1, C28.1, U$18.2, U$2.VIN+
- new net -15V: -15V.TST_POINT, U$18.3
- new net -9V_F_DUAL: C14.2, C16.2, C17.2, U$13.IN, U$5.3
- new net -9V_UF: -9V_U.TST_POINT, C18.1, C19.1, L2.1, L2_CUK.1, R7.2
- new net 5V_REF: C29.1, C30.1, C6.1, R12.2, R9.2, U$20.VOUT, U$6.REF, VREF.TST_POINT
- new net 9V_F_DUAL: C13.1, C15.1, C17.1, U$12.OUT, U$5.2
- new net 9V_F_SINGLE: 9V_F_S.TST_POINT, C3.1, C31.1, C4.1, T2.C, U$15.OUT, U$17.EN, U$17.VIN, U$1G$3.V+, U$20.VIN
- new net 9V_UF: 9V_UF.TST_POINT, C21.1, L1.1, L1_CUK.2, L3.1, U$2.VOUT+, U$7./SHDN, U$7.VIN
- new net 9V_UF1: C1.1, C2.1, L3.2, U$14.IN_HIGH
- new net D_GND: C25.1, U$19.2
- new net GND_ISO_UF: C1.2, C10.2, C11.2, C12.2, C18.2, C2.2, C21.2, C9.2, GND_ISO_UF.TST_POINT, R8.1, U$10.C, U$14.IN_LOW, U$2.VOUT-, U$7.GND
- new net N$11: C19.2, R7.1, R8.2, U$7.NFB
- new net N$12: C20.1, L1_CUK.1, U$7.SW
- new net N$13: U$11.OUT_HIGH, U$12.IN
- new net N$14: U$11.OUT_LOW, U$13.OUT
- new net N$15: C20.2, L2_CUK.2, U$10.A
- new net N$16: C11.1, C12.1, L2.2, U$11.IN_LOW
- new net N$17: U$14.OUT_HIGH, U$15.IN
- new net N$18: R6.1, U$1G$1.AIN+, U$3.COMMON
- new net N$2: R10.1, R9.1
- new net N$5: C22.1, U$17.NR
- new net N$6: C10.1, C9.1, L1.2, U$11.IN_HIGH
- new net SCL: R14.1, U$19.3, U$4.SCL, U$6.SCL
- new net SDA: R13.1, U$19.4, U$4.SDA, U$6.SDA
- new net V_SENSE: C8.1, R1.1, R2.2, U$4.VIN+
- net 5V: now also 5V.TST_POINT, C23.1, C24.1, C5.1, C7.1, R13.2, R14.2, U$17.OUT, U$4.VDD, U$6.AUX, U$6.VDD; no longer RREF.2
- net GND_ISO: now also C13.2, C14.1, C15.2, C16.1, C22.2, C23.2, C24.2, C25.2, C29.2, C3.2, C30.2, C31.2, C4.2, C5.2, C6.2, C7.2, C8.2, GND_ISO.TST_POINT, R10.2, R11.1, R2.1, R3.1, R6.2, U$12.GND, U$13.GND, U$14.OUT_LOW, U$15.GND, U$16.1, U$17.GND, U$20.GND, U$4.VIN-, U$4.VSS, U$5.1, U$5.4, U$6.ADDR, U$6.GND; no longer REF_POT.2, REF_POT.W, RFB2.1, U$2.VOUT-
- net INST_GND: now also C26.2, C27.2, C28.2, U$18.1, U$18.4
- net N$3: now also R5.2; no longer RLIMIT.2
- net REF1: now also R10.W; no longer REF_POT.1, RREF.1
- net REF2: now also U$6.OUT
- net REF3: now also R11.2, R12.1
- net VADJ: now also R1.2, R4.2, R5.1, U$16.2; no longer RFB1.2, RLIMIT.1
- net VFB: now also R3.2, R4.1; no longer RFB1.1, RFB2.2
Other:
- note added: "1uF"
- note added: "ADJUSTABLE REGULATOR FOR TEC"
- note added: "DATA INPUT (I2C)"
- note added: "DIVIDE THIS DOWN FURTHER!!!"
- note added: "FZT653CT"
- note added: "INSTRUMENT POWER INPUT"
- note added: "LMC6482"
- note added: "LT1461"
- note added: "MCP3425"
- note added: "MMBT3904"
- note added: "PRE AMP VOLTAGE REGULATION"
- note added: "PREAMP OUTPUT"
- note added: "REC7.5"
- note added: "REFERENCES"
- note added: "REG102"
- note added: "SYSTEM POWER"
- note added: "TEC OUTPUT"

Commit message: Layout mostly complete. Making finishing documentation touches:
Parts:
- J1, J2, J3: value 4-OUT -> (none)
- J4: value 2-THRU -> (none)
- T2: value FZT653-NPNBJT -> (none)
- renumbered L1_CUK to L6, L2_CUK to L7, U$1 to U1, U$11 to L4, U$12 to FC2, U$13 to FC1, U$14 to L5, U$15 to FC3, U$16 to J4, U$17 to U5, U$18 to J1, U$19 to J3, U$2 to U4, U$20 to U3, U$4 to U6, U$5 to J2, U$6 to U2, U$7 to U7
